Commit message: fix broken gripper 2f 85 robotiq/issues/150

File: robotiq_2f_85_gripper_visualization/urdf/robotiq_arg2f_transmission.xacro (robot description, xacro)
@@ -11,4 +11,39 @@
       </actuator>
     </transmission>
+    <!-- To fix broken gripper in gazebo according to the following issue-->
+    <!--https://github.com/ros-industrial/robotiq/issues/150-->
+    <gazebo>
+             <!-- loading plugin: mimic joints works in gazebo now-->
+             <plugin filename="libroboticsgroup_gazebo_mimic_joint_plugin.so" name="${prefix}mimic_robotiq_85_4">
+                <joint>${prefix}finger_joint</joint>
+                <mimicJoint>${prefix}right_outer_knuckle_joint</mimicJoint>
+                <!--<multiplier>-1.0</multiplier>-->
+                <!--<offset>0.0</offset>-->
+            </plugin>
+            <plugin filename="libroboticsgroup_gazebo_mimic_joint_plugin.so" name="${prefix}mimic_robotiq_85_2">
+                <joint>${prefix}finger_joint</joint>
+                <mimicJoint>${prefix}left_inner_finger_joint</mimicJoint>
+                <!--<multiplier>1.0</multiplier>-->
+                <!--<offset>0.0</offset>-->
+            </plugin>
+            <plugin filename="libroboticsgroup_gazebo_mimic_joint_plugin.so" name="${prefix}mimic_robotiq_85_6">
+                <joint>${prefix}finger_joint</joint>
+                <mimicJoint>${prefix}right_inner_finger_joint</mimicJoint>
+                <!--<multiplier>1.0</multiplier>-->
+                <!--<offset>0.0</offset>-->
+            </plugin>
+            <plugin filename="libroboticsgroup_gazebo_mimic_joint_plugin.so" name="${prefix}mimic_robotiq_85_3">
+                <joint>${prefix}finger_joint</joint>
+                <mimicJoint>${prefix}left_inner_knuckle_joint</mimicJoint>
+                <!--<multiplier>-1.0</multiplier>-->
+                <!--<offset>0.0</offset>-->
+            </plugin>
+            <plugin filename="libroboticsgroup_gazebo_mimic_joint_plugin.so" name="${prefix}mimic_robotiq_85_5">
+                <joint>${prefix}finger_joint</joint>
+                <mimicJoint>${prefix}right_inner_knuckle_joint</mimicJoint>
+                <!--<multiplier>-1.0</multiplier>-->
+                <!--<offset>0.0</offset>-->
+            </plugin>
+        </gazebo>
   </xacro:macro>
 </robot>

Commit message: robotiq 85 : gazebo mimic joint specific file

File: robotiq_2f_85_gripper_visualization/urdf/robotiq_arg2f_transmission.xacro (robot description, xacro)
@@ -5,5 +5,6 @@
       <type>transmission_interface/SimpleTransmission</type>
       <joint name="${prefix}finger_joint">
-        <hardwareInterface>hardware_interface/PositionJointInterface</hardwareInterface>
+        <hardwareInterface>hardware_interface/EffortJointInterface</hardwareInterface>
+        <!--<hardwareInterface>hardware_interface/PositionJointInterface</hardwareInterface>-->
       </joint>
       <actuator name="${prefix}finger_joint_motor">
@@ -11,39 +12,6 @@
       </actuator>
     </transmission>
-    <!-- To fix broken gripper in gazebo according to the following issue-->
-    <!--https://github.com/ros-industrial/robotiq/issues/150-->
-    <gazebo>
-             <!-- loading plugin: mimic joints works in gazebo now-->
-             <plugin filename="libroboticsgroup_gazebo_mimic_joint_plugin.so" name="${prefix}mimic_robotiq_85_4">
-                <joint>${prefix}finger_joint</joint>
-                <mimicJoint>${prefix}right_outer_knuckle_joint</mimicJoint>
-                <!--<multiplier>-1.0</multiplier>-->
-                <!--<offset>0.0</offset>-->
-            </plugin>
-            <plugin filename="libroboticsgroup_gazebo_mimic_joint_plugin.so" name="${prefix}mimic_robotiq_85_2">
-                <joint>${prefix}finger_joint</joint>
-                <mimicJoint>${prefix}left_inner_finger_joint</mimicJoint>
-                <!--<multiplier>1.0</multiplier>-->
-                <!--<offset>0.0</offset>-->
-            </plugin>
-            <plugin filename="libroboticsgroup_gazebo_mimic_joint_plugin.so" name="${prefix}mimic_robotiq_85_6">
-                <joint>${prefix}finger_joint</joint>
-                <mimicJoint>${prefix}right_inner_finger_joint</mimicJoint>
-                <!--<multiplier>1.0</multiplier>-->
-                <!--<offset>0.0</offset>-->
-            </plugin>
-            <plugin filename="libroboticsgroup_gazebo_mimic_joint_plugin.so" name="${prefix}mimic_robotiq_85_3">
-                <joint>${prefix}finger_joint</joint>
-                <mimicJoint>${prefix}left_inner_knuckle_joint</mimicJoint>
-                <!--<multiplier>-1.0</multiplier>-->
-                <!--<offset>0.0</offset>-->
-            </plugin>
-            <plugin filename="libroboticsgroup_gazebo_mimic_joint_plugin.so" name="${prefix}mimic_robotiq_85_5">
-                <joint>${prefix}finger_joint</joint>
-                <mimicJoint>${prefix}right_inner_knuckle_joint</mimicJoint>
-                <!--<multiplier>-1.0</multiplier>-->
-                <!--<offset>0.0</offset>-->
-            </plugin>
-        </gazebo>
+  <!--Gazebo mimic joints-->
+  <xacro:include filename="$(find robotiq_2f_85_gripper_visualization)/urdf/robotiq_arg2f_85.gazebo.xacro" />
   </xacro:macro>
 </robot>
