Commit message: added dummy base link

File: robotiq_2f_85_gripper_visualization/urdf/robotiq_arg2f_85_macro.xacro (robot description, xacro)
@@ -180,4 +180,9 @@
     </xacro:macro>
     <!-- base link -->
+    <link name="${prefix}base_link"/>
+    <joint name="${prefix}base_link-${prefix}robotiq_arg2f_base_link" type="fixed">
+      <parent link="${prefix}base_link" />
+      <child link="${prefix}robotiq_arg2f_base_link" />
+    </joint>
     <link name="${prefix}robotiq_arg2f_base_link">
         <inertial>

Commit message: Add a TCP fixed joint

File: robotiq_2f_85_gripper_visualization/urdf/robotiq_arg2f_85_macro.xacro (robot description, xacro)
@@ -206,4 +206,11 @@
         </collision>
       </link>
+    <!-- TCP frame centered between the fingers near the grasp equilibrium point -->
+    <link name="${prefix}robotiq_arg2f_tcp"/>
+    <joint name="${prefix}robotiq_arg2f_tcp_joint" type="fixed">
+      <origin rpy="0 0 0" xyz="0 0 0.174"/>
+      <parent link="${prefix}robotiq_arg2f_base_link"/>
+      <child link="${prefix}robotiq_arg2f_tcp"/>
+    </joint>
     <!-- left finger -->
     <xacro:finger_links prefix="${prefix}" fingerprefix="left"/>

Commit message: Update masses based on OnShape checks

File: robotiq_2f_85_gripper_visualization/urdf/robotiq_arg2f_85_macro.xacro (robot description, xacro)
@@ -13,5 +13,5 @@
         <inertial>
           <origin xyz="-0.000200000000003065 0.0199435877845359 0.0292245259211331" rpy="0 0 0" />
-          <mass value="0.00853198276973456" />
+          <mass value="0.013" />
           <inertia ixx="2.89328108496468E-06" ixy="-1.57935047237397E-19" ixz="-1.93980378593255E-19" iyy="1.86719750325683E-06" iyz="-1.21858577871576E-06" izz="1.21905238907251E-06" />
           </inertial>
@@ -37,5 +37,5 @@
         <inertial>
           <origin xyz="0.00030115855001899 0.0373907951953854 -0.0208027427000385" rpy="0 0 0" />
-          <mass value="0.022614240507152" />
+          <mass value="0.041" />
           <inertia ixx="1.52518312458174E-05" ixy="9.76583423954399E-10" ixz="-5.43838577022588E-10" iyy="6.17694243867776E-06" iyz="6.78636130740228E-06" izz="1.16494917907219E-05" />
           </inertial>
@@ -61,5 +61,5 @@
         <inertial>
           <origin xyz="0.000123011831763771 0.0507850843201817 0.00103968640075166" rpy="0 0 0" />
-        <mass value="0.0271177346495152" />
+        <mass value="0.028" />
           <inertia ixx="2.61910379223783E-05" ixy="-2.43616858946494E-07" ixz="-6.37789906117123E-09" iyy="2.8270243746167E-06" iyz="-5.37200748039765E-07" izz="2.83695868220296E-05" />
           </inertial>
@@ -85,5 +85,5 @@
         <inertial>
           <origin xyz="0.000299999999999317 0.0160078233491243 -0.0136945669206257" rpy="0 0 0" />
-          <mass value="0.0104003125914103" />
+          <mass value="0.04" />
           <inertia ixx="2.71909453810972E-06" ixy="1.35402465472579E-21" ixz="-7.1817349065269E-22" iyy="7.69100314106116E-07" iyz="6.74715432769696E-07" izz="2.30315190420171E-06" />
           </inertial>
@@ -187,6 +187,6 @@
         <inertial>
           <origin xyz="8.625E-08 -4.6583E-06 0.03145" rpy="0 0 0" />
-          <mass value="0.7" />
-          <inertia ixx="0.00020005" ixy="-4.2442E-10" ixz="-2.9069E-10" iyy="0.00017832" iyz="-3.4402E-08" izz="0.00013478" />
+          <mass value="0.635" />
+          <inertia ixx="0.000494023" ixy="0.0" ixz="0.0" iyy="0.000562779" iyz="0.0" izz="0.000377692" />
         </inertial>
         <visual>

Commit message: Add newer overmolded fingertip model

File: robotiq_2f_85_gripper_visualization/urdf/robotiq_arg2f_85_macro.xacro (robot description, xacro)
@@ -22,5 +22,5 @@
           </geometry>
           <material name="">
-            <color rgba="0.792156862745098 0.819607843137255 0.933333333333333 1" />
+            <color rgba="0.65 0.65 0.65 1" />
           </material>
         </visual>
@@ -46,5 +46,5 @@
           </geometry>
           <material name="">
-            <color rgba="0.1 0.1 0.1 1" />
+            <color rgba="0.13 0.13 0.13 1" />
           </material>
         </visual>
@@ -70,5 +70,5 @@
           </geometry>
           <material name="">
-            <color rgba="0.1 0.1 0.1 1" />
+            <color rgba="0.13 0.13 0.13 1" />
           </material>
         </visual>
@@ -84,53 +84,51 @@
       <link name="${prefix}${fingerprefix}_distal_phalanx">
         <inertial>
-          <origin xyz="0.000299999999999317 0.0160078233491243 -0.0136945669206257" rpy="0 0 0" />
-          <mass value="0.04" />
-          <inertia ixx="2.71909453810972E-06" ixy="1.35402465472579E-21" ixz="-7.1817349065269E-22" iyy="7.69100314106116E-07" iyz="6.74715432769696E-07" izz="2.30315190420171E-06" />
-          </inertial>
-        <visual>
-          <origin xyz="0 0 0" rpy="0 0 0" />
-          <geometry>
-            <mesh filename="package://robotiq_2f_85_gripper_visualization/meshes/visual/distal_phalanx.stl" />
-          </geometry>
-          <material name="">
-            <color rgba="0.1 0.1 0.1 1" />
-          </material>
-        </visual>
-        <collision>
-          <origin xyz="0 0 0" rpy="0 0 0" />
-          <geometry>
-            <mesh filename="package://robotiq_2f_85_gripper_visualization/meshes/collision/distal_phalanx.stl" />
-          </geometry>
-        </collision>
-      </link>
-    </xacro:macro>
-    <!-- Finger pad link, the default are the "big pads" with rubber-->
-    <!-- <xacro:macro name="pad" params="prefix fingerprefix">
-      <link name="${prefix}${fingerprefix}_pad">
-        <visual>
-          <origin xyz="0 0 0" rpy="0 0 0" />
-          <geometry>
-            <box size="0.022 0.00635 0.0375"/>
-          </geometry>
-          <material name="">
-            <color rgba="0.9 0.9 0.9 1" />
-          </material>
-        </visual>
-        <collision>
-          <origin xyz="0 0 0" rpy="0 0 0" />
-          <geometry>
-            <box size="0.022 0.00635 0.0375"/>
-          </geometry>
-          <material name="">
-            <color rgba="0.9 0.0 0.0 1" />
-          </material>
-        </collision>
-      </link>
-    </xacro:macro> -->
+          <origin xyz="0 -0.009 0.005" rpy="0 0 0" />
+          <mass value="0.02" />
+          <inertia ixx="1.839e-6" ixy="2.943e-15" ixz="-8.887e-15" iyy="1.184e-6" iyz="4.328e-7" izz="1.820e-6" />
+          </inertial>
+        <visual>
+          <origin xyz="0 0 0" rpy="0 0 0" />
+          <geometry>
+            <mesh filename="package://robotiq_2f_85_gripper_visualization/meshes/visual/driver.dae" />
+          </geometry>
+          <material name="">
+            <color rgba="0.13 0.13 0.13 1" />
+          </material>
+        </visual>
+        <collision>
+          <origin xyz="0 0 0" rpy="0 0 0" />
+          <geometry>
+            <mesh filename="package://robotiq_2f_85_gripper_visualization/meshes/collision/driver.stl" />
+          </geometry>
+        </collision>
+      </link>
+    </xacro:macro>
+    <xacro:macro name="finger_tip" params="prefix fingerprefix">
+      <link name="${prefix}${fingerprefix}_finger_tip">
+        <inertial>
+          <origin xyz="0 -0.008 0.016" rpy="0 0 0" />
+          <mass value="0.021" />
+          <inertia ixx="3.071e-6" ixy="-3.735e-13" ixz="-1.785e-13" iyy="3.467e-6" iyz="4.052e-7" izz="1.175e-6" />
+        </inertial>
+        <visual>
+          <origin xyz="0 0 0" rpy="0 0 0" />
+          <geometry>
+            <mesh filename="package://robotiq_2f_85_gripper_visualization/meshes/visual/agc-tip-mld-kit-85.dae" />
+          </geometry>
+        </visual>
+        <collision>
+          <origin xyz="0 0 0" rpy="0 0 0" />
+          <geometry>
+            <mesh filename="package://robotiq_2f_85_gripper_visualization/meshes/collision/agc-tip-mld-kit-85.stl" />
+          </geometry>
+        </collision>
+      </link>
+    </xacro:macro>
     <xacro:macro name="finger_links" params="prefix fingerprefix">
       <xacro:outer_knuckle prefix="${prefix}" fingerprefix="${fingerprefix}"/>
       <xacro:bar prefix="${prefix}" fingerprefix="${fingerprefix}"/>
       <xacro:distal_phalanx prefix="${prefix}" fingerprefix="${fingerprefix}"/>
-      <!-- <xacro:pad prefix="${prefix}" fingerprefix="${fingerprefix}"/> -->
+      <xacro:finger_tip prefix="${prefix}" fingerprefix="${fingerprefix}"/>
       <xacro:proximal_phalanx prefix="${prefix}" fingerprefix="${fingerprefix}"/>
     </xacro:macro>
@@ -164,16 +162,16 @@
       </joint>
     </xacro:macro>
-    <!-- <xacro:macro name="pad_joint" params="prefix fingerprefix">
-      <joint name="${prefix}${fingerprefix}_pad_joint" type="fixed">
-        <origin xyz="0 -0.0220203446692936 0.03242" rpy="0 0 0"/>
+    <xacro:macro name="finger_tip_joint" params="prefix fingerprefix">
+      <joint name="${prefix}${fingerprefix}_finger_tip_joint" type="fixed">
+        <origin xyz="0 -0.011402 0.01305" rpy="0 0 0"/>
         <parent link="${prefix}${fingerprefix}_distal_phalanx" />
-        <child link="${prefix}${fingerprefix}_pad" />
-        <axis xyz="0 0 1" />
-      </joint>
-    </xacro:macro> -->
+        <child link="${prefix}${fingerprefix}_finger_tip" />
+      </joint>
+    </xacro:macro>
     <xacro:macro name="finger_joints" params="prefix fingerprefix reflect">
       <xacro:bar_joint prefix="${prefix}" fingerprefix="${fingerprefix}"/>
       <xacro:proximal_phalanx_joint prefix="${prefix}" fingerprefix="${fingerprefix}" reflect="${reflect}"/>
       <xacro:distal_phalanx_joint prefix="${prefix}" fingerprefix="${fingerprefix}"/>
+      <xacro:finger_tip_joint prefix="${prefix}" fingerprefix="${fingerprefix}"/>
       <!-- <xacro:pad_joint prefix="${prefix}" fingerprefix="${fingerprefix}"/> -->
     </xacro:macro>
@@ -196,5 +194,5 @@
           </geometry>
           <material name="">
-            <color rgba="0.1 0.1 0.1 1" />
+            <color rgba="0.13 0.13 0.13 1" />
           </material>
         </visual>
