Commit message: removed gazebo reference from here, renamed macro, introduced hw_interfce arg

File: robotiq_2f_85_gripper_visualization/urdf/inc/robotiq_arg2f_85_transmissions.xacro (robot description, xacro)
@@ -1,10 +1,9 @@
 <?xml version="1.0"?>
 <robot xmlns:xacro="http://ros.org/wiki/xacro">
-  <xacro:macro name="robotiq_arg2f_transmission" params="prefix">
+  <xacro:macro name="robotiq_arg2f_85_transmission" params="prefix hw_interface">
     <transmission name="${prefix}finger_joint_trans">
       <type>transmission_interface/SimpleTransmission</type>
       <joint name="${prefix}finger_joint">
-        <hardwareInterface>hardware_interface/EffortJointInterface</hardwareInterface>
-        <!--<hardwareInterface>hardware_interface/PositionJointInterface</hardwareInterface>-->
+        <hardwareInterface>${hw_interface}</hardwareInterface>
       </joint>
       <actuator name="${prefix}finger_joint_motor">
@@ -12,6 +11,4 @@
       </actuator>
     </transmission>
-  <!--Gazebo mimic joints-->
-  <xacro:include filename="$(find robotiq_2f_85_gripper_visualization)/urdf/robotiq_arg2f_85.gazebo.xacro" />
   </xacro:macro>
 </robot>
